File: PCB/Actuators.kicad_sch (KiCad schematic)
At the start: 90 parts, among them J1 R_Motor, J10 Servos, J11 PWR-Servos, J3 Left_Speaker, J4 Right_Speaker, J5 GAIN_sel, J6 R_Motor, J7 Servos, J8 Servos, J9 Servos, Q1 AOD417, U10 BTN7960B, U11 PCA9685PW, U2 MAX98357A, U4 MAX98357A, U5 BTN7960B, U6 BTN7960B, U7 74HC244, U8 74HC244, U9 BTN7960B

Commit message: [Schem] Finished the whole Schematic (Connected all the pins)
Connections:
- net OE: no longer names the net of R40.1, U11.23 (~{OE})
Changed lines of the file:
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@@
-		)
-	)
-	(hierarchical_label "OE"
-		(shape input)
-		(at 72.39 157.48 270)
-		(effects
-			(font
-				(size 1.27 1.27)
-				(thickness 0.254)
-				(bold yes)
-			)
-			(justify right)
 		)
 	)
@@
 		(in_pos_files yes)
 		(dnp no)
-		(fields_autoplaced yes)
 		(property "Reference" "C20"
 			(at 55.88 74.9299 0)
@@
 		)
 		(property "Value" "0.1 uF"
-			(at 55.88 77.4699 0)
-			(show_name no)
-			(do_not_autoplace no)
+			(at 54.864 76.708 0)
+			(show_name no)
+			(do_not_autoplace no)
