File: PCB/Actuators.kicad_sch (KiCad schematic)
At the start: 82 parts, among them J1 R_Motor, J10 Servos, J3 Left_Speaker, J4 Right_Speaker, J5 GAIN_sel, J6 L_Motor, J7 Servos, J8 Servos, J9 Servos, Q1 AOD417, U10 BTN7960B, U11 PCA9685PW, U2 MAX98357A, U4 MAX98357A, U5 BTN7960B, U6 BTN7960B, U7 74HC244, U8 74HC244, U9 BTN7960B

Commit message: [PCB] Splited the PCB into two boards
Connections:
- net +5V: no longer C1.1, C22.1, C25.1, D7.2 (A), R57.1, R58.1, U11.1 (A0), U11.28 (VDD), U7.20 (VCC), U8.20 (VCC)
- new net +5VCo: C1.1, C22.1, C25.1, D7.2 (A), R57.1, R58.1, U11.1 (A0), U11.28 (VDD), U7.20 (VCC), U8.20 (VCC)
Changed lines of the file:
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@@
 		(in_pos_files yes)
 		(dnp no)
-		(fields_autoplaced yes)
 		(property "Reference" "#PWR030"
 			(at 200.66 25.4 0)
@@
 			)
 		)
-		(property "Value" "+5V"
-			(at 200.66 16.51 0)
+		(property "Value" "+5VCo"
+			(at 203.2 20.3199 0)
 			(show_name no)
 			(do_not_autoplace no)
@@
 					(size 1.27 1.27)
 				)
+				(justify left)
 			)
 		)
@@
 		(in_pos_files yes)
 		(dnp no)
-		(fields_autoplaced yes)
 		(property "Reference" "#PWR085"
 			(at 73.66 137.16 0)
@@
 			)
 		)
-		(property "Value" "+5V"
-			(at 73.66 128.27 0)
+		(property "Value" "+5VCo"
+			(at 70.104 128.778 0)
 			(show_name no)
 			(do_not_autoplace no)
@@
 					(size 1.27 1.27)
 				)
+				(justify left)
 			)
 		)
@@
 		(in_pos_files yes)
 		(dnp no)
-		(fields_autoplaced yes)
 		(property "Reference" "#PWR084"
 			(at 30.48 160.02 0)
@@
 			)
 		)
-		(property "Value" "+5V"
-			(at 30.48 151.13 0)
+		(property "Value" "+5VCo"
+			(at 27.432 151.892 0)
 			(show_name no)
 			(do_not_autoplace no)
@@
 					(size 1.27 1.27)
 				)
+				(justify left)
 			)
 		)
@@
 		(in_pos_files yes)
 		(dnp no)
-		(fields_autoplaced yes)
 		(property "Reference" "#PWR083"
 			(at 95.25 133.35 0)
@@
 			)
 		)
-		(property "Value" "+5V"
-			(at 95.25 124.46 0)
+		(property "Value" "+5VCo"
+			(at 91.44 124.968 0)
 			(show_name no)
 			(do_not_autoplace no)
@@
 					(size 1.27 1.27)
 				)
+				(justify left)
 			)
 		)
@@
 		(in_pos_files yes)
 		(dnp no)
-		(fields_autoplaced yes)
 		(property "Reference" "#PWR035"
 			(at 370.84 26.67 0)
@@
 			)
 		)
-		(property "Value" "+5V"
-			(at 370.84 17.78 0)
+		(property "Value" "+5VCo"
+			(at 373.38 21.5899 0)
 			(show_name no)
 			(do_not_autoplace no)
@@
 					(size 1.27 1.27)
 				)
+				(justify left)
 			)
 		)
