File: PCB/Brain.kicad_sch (KiCad schematic)
At the start: 1 part, among them J14 Raspberry_Pi_Zero

Commit message: [Schem] Finished the whole Schematic (Connected all the pins)
Other:
- sheet ESP32-S3 ports: added none; removed 0RX, 0TX
Changed lines of the file:
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@@
-		)
-	)
-	(hierarchical_label "0TX"
-		(shape bidirectional)
-		(at 115.57 76.2 0)
-		(effects
-			(font
-				(size 1.27 1.27)
-			)
-			(justify left)
 		)
 	)
@@
 			)
 			(justify right)
-		)
-	)
-	(hierarchical_label "0RX"
-		(shape bidirectional)
-		(at 115.57 78.74 0)
-		(effects
-			(font
-				(size 1.27 1.27)
-			)
-			(justify left)
 		)
 	)
@@
 			)
 		)
-		(pin "0RX" input
-			(at 115.57 78.74 0)
-			(effects
-				(font
-					(size 1.27 1.27)
-				)
-				(justify right)
-			)
-		)
 		(pin "GPIO0" bidirectional
 			(at 115.57 114.3 0)
@@
 			)
 		)
-		(pin "ESP_3v3" output
+		(pin "ESP_3v3" input
 			(at 87.63 76.2 180)
 			(effects
@@
 			(effects
 				(font
-					(size 1.27 1.27)
-				)
-				(justify right)
-			)
-		)
-		(pin "0TX" output
-			(at 115.57 76.2 0)
-			(effects
-				(font
