File: PCB/ESP32-S3.kicad_sch (KiCad schematic)
At the start: 30 parts, among them J2 USB_C_Receptacle_USB2.0_16P, SW1 SW_MEC_5E, SW2 SW_MEC_5E, SW3 SW_MEC_5E, U1 ESP32-S3-WROOM-1, U3 AMS1117-3.3

Commit message: [Schem] Finished the whole Schematic (Connected all the pins)
Parts:
- added J13: Debug, symbol Connector_Generic:Conn_01x04
Connections:
- net +3.3V: now also J13.4 (Pin_4)
- net 0RX: now also J13.2 (Pin_2)
- net 0TX: now also J13.1 (Pin_1)
- net GND: now also J13.3 (Pin_3)
