File: PCB/sensors.kicad_sch (KiCad schematic)
At the start: 0 parts

Commit message: [Schem] Added sensors connectors & finished Step down circuit
Parts:
- added J12: R-INMP441, symbol Connector_Generic:Conn_02x03_Counter_Clockwise
- added J13: L-INMP441, symbol Connector_Generic:Conn_02x03_Counter_Clockwise
- added J15: F_HS-SR04+, symbol Connector_Generic:Conn_01x04
- added J16: B_HS-SR04+, symbol Connector_Generic:Conn_01x04
- added J17: MPU-6050, symbol Connector_Generic:Conn_01x08
- added U12: Module-3, symbol WALL-E_symbols:Camera
Connections:
- new net +3.3V: J12.1 (Pin_1), J12.5 (Pin_5), J13.5 (Pin_5), J15.1 (Pin_1), J16.1 (Pin_1), J17.1 (Pin_1)
- new net B_Echo: J16.3 (Pin_3)
- new net B_Trig: J16.2 (Pin_2)
- new net F_Echo: J15.3 (Pin_3)
- new net F_Trig: J15.2 (Pin_2)
- new net GND: J12.4 (Pin_4), J13.1 (Pin_1), J13.4 (Pin_4), J15.4 (Pin_4), J16.4 (Pin_4), J17.2 (Pin_2)
- new net L-mic_SCK: J13.3 (Pin_3)
- new net L-mic_SD: J13.6 (Pin_6)
- new net L-mic_WS: J13.2 (Pin_2)
- new net R-mic_SCK: J12.3 (Pin_3)
- new net R-mic_SD: J12.6 (Pin_6)
- new net R-mic_WS: J12.2 (Pin_2)
- new net SCL: J17.3 (Pin_3)
- new net SDA: J17.4 (Pin_4)
- no-connect marks 0 -> 4

Commit message: [Schem] Added all the net labels and connected the Dashboard screen
Connections:
- net SCL renamed Mot_SCL
- net SDA renamed Mot_SDA
Changed lines of the file:
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@@
 	(wire
 		(pts
-			(xy 120.65 109.22) (xy 110.49 109.22)
+			(xy 111.76 105.41) (xy 110.49 105.41)
 		)
 		(stroke
@@
 	(wire
 		(pts
+			(xy 111.76 105.41) (xy 111.76 109.22)
+		)
+		(stroke
+			(width 0)
+			(type default)
+		)
+	)
+	(wire
+		(pts
 			(xy 119.38 114.3) (xy 120.65 114.3)
 		)
@@
 	(wire
 		(pts
+			(xy 111.76 109.22) (xy 120.65 109.22)
+		)
+		(stroke
+			(width 0)
+			(type default)
+		)
+	)
+	(wire
+		(pts
 			(xy 190.5 82.55) (xy 193.04 82.55)
 		)
@@
 		)
 	)
-	(hierarchical_label "SCL"
+	(hierarchical_label "Mot_SCL"
 		(shape input)
 		(at 119.38 111.76 180)
@@
 		)
 	)
-	(hierarchical_label "SDA"
+	(hierarchical_label "Mot_SDA"
 		(shape input)
 		(at 119.38 114.3 180)
@@
 	(symbol
 		(lib_id "power:GND")
-		(at 110.49 109.22 0)
+		(at 110.49 105.41 0)
 		(unit 1)
 		(body_style 1)
@@
 		(in_pos_files yes)
 		(dnp no)
-		(fields_autoplaced yes)
 		(property "Reference" "#PWR0117"
-			(at 110.49 115.57 0)
+			(at 110.49 111.76 0)
 			(hide yes)
 			(show_name no)
@@
 		)
 		(property "Value" "GND"
-			(at 110.49 114.3 0)
+			(at 110.49 109.22 0)
 			(show_name no)
 			(do_not_autoplace no)
@@
 		)
 		(property "Footprint" ""
-			(at 110.49 109.22 0)
+			(at 110.49 105.41 0)
 			(hide yes)
 			(show_name no)
@@
 		)
 		(property "Datasheet" ""
-			(at 110.49 109.22 0)
+			(at 110.49 105.41 0)
 			(hide yes)
 			(show_name no)
@@
 		)
 		(property "Description" "Power symbol creates a global label with name \"GND\" , ground"
-			(at 110.49 109.22 0)
-			(hide yes)
-			(show_name no)
+			(at 110.49 105.41 0)
+			(hide yes)
+			(show_name no)

Commit message: [PCB] Assigned all the footprints
Parts:
- removed J13: L-INMP441, symbol Connector_Generic:Conn_02x03_Counter_Clockwise
- J12: footprint (none) -> Connector_JST:JST_ZH_B6B-ZR-SM4-TF_1x06-1MP_P1.50mm_Vertical
- J15, J16: footprint (none) -> Connector_JST:JST_ZH_B4B-ZR-SM4-TF_1x04-1MP_P1.50mm_Vertical
- J17: footprint (none) -> Connector_JST:JST_ZH_B8B-ZR-SM4-TF_1x08-1MP_P1.50mm_Vertical
Connections:
- net R-mic_SCK renamed mic_SCK
- net R-mic_SD renamed mic_SD
- net R-mic_WS renamed mic_WS
Other:
- moved on the sheet: J12

Commit message: [PCB] 95% finished the PCB
Parts:
- J12: value R-INMP441 -> L-INMP441
Connections:
- net +3.3V: no longer J12.1 (Pin_1)
- net GND: now also J12.1 (Pin_1)
Changed lines of the file:
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@@
+	(wire
+		(pts
+			(xy 104.14 74.93) (xy 106.68 74.93)
+		)
+		(stroke
+			(width 0)
+			(type default)
+		)
+	)
 	(wire
 		(pts
@@
 	(wire
 		(pts
+			(xy 104.14 74.93) (xy 104.14 76.2)
+		)
+		(stroke
+			(width 0)
+			(type default)
+		)
+	)
+	(wire
+		(pts
 			(xy 139.7 83.82) (xy 124.46 83.82)
 		)
@@
 	(wire
 		(pts
+			(xy 106.68 81.28) (xy 111.76 81.28)
+		)
+		(stroke
+			(width 0)
+			(type default)
+		)
+	)
+	(wire
+		(pts
 			(xy 166.37 83.82) (xy 167.64 83.82)
 		)
@@
 	(wire
 		(pts
-			(xy 111.76 81.28) (xy 107.95 81.28)
+			(xy 106.68 74.93) (xy 106.68 81.28)
 		)
 		(stroke
@@
 	)
 	(symbol
+		(lib_id "power:GND")
+		(at 104.14 76.2 0)
+		(unit 1)
+		(body_style 1)
+		(exclude_from_sim no)
+		(in_bom yes)
+		(on_board yes)
+		(in_pos_files yes)
+		(dnp no)
+		(fields_autoplaced yes)
+		(property "Reference" "#PWR0112"
+			(at 104.14 82.55 0)
+			(hide yes)
+			(show_name no)
+			(do_not_autoplace no)
+			(effects
+				(font
+					(size 1.27 1.27)
+				)
+			)
+		)
+		(property "Value" "GND"
+			(at 104.14 81.28 0)
+			(show_name no)
+			(do_not_autoplace no)
+			(effects
+				(font
+					(size 1.27 1.27)
+				)
+			)
+		)
+		(property "Footprint" ""
+			(at 104.14 76.2 0)
+			(hide yes)
+			(show_name no)
+			(do_not_autoplace no)
+			(effects
+				(font
+					(size 1.27 1.27)
+				)
+			)
+		)
+		(property "Datasheet" ""
+			(at 104.14 76.2 0)
+			(hide yes)
+			(show_name no)
+			(do_not_autoplace no)
+			(effects
+				(font
+					(size 1.27 1.27)
+				)
+			)
+		)
+		(property "Description" "Power symbol creates a global label with name \"GND\" , ground"
+			(at 104.14 76.2 0)
+			(hide yes)
+			(show_name no)
+			(do_not_autoplace no)
+			(effects
+				(font
+					(size 1.27 1.27)
+				)
+			)
+		)
+		(pin "1"
+		)
+		(instances
+			(project "PCB"
+				(path "/ce714510-8789-438c-9780-97c7c26e78af/77c81cbd-c586-4d65-a39c-d5337f0031c1"
+					(reference "#PWR0112")
+					(unit 1)
+				)
+			)
+		)
+	)
+	(symbol
 		(lib_id "power:+3.3V")
 		(at 165.1 78.74 0)
@@
 				(path "/ce714510-8789-438c-9780-97c7c26e78af/77c81cbd-c586-4d65-a39c-d5337f0031c1"
 					(reference "#PWR0114")
-					(unit 1)
-				)
-			)
-		)
-	)
-	(symbol
-		(lib_id "power:+3.3V")
-		(at 107.95 81.28 0)
-		(unit 1)
-		(body_style 1)
-		(exclude_from_sim no)
-		(in_bom yes)
-		(on_board yes)
-		(in_pos_files yes)
-		(dnp no)
-		(fields_autoplaced yes)
-		(property "Reference" "#PWR0107"
-			(at 107.95 85.09 0)
-			(hide yes)
-			(show_name no)
-			(do_not_autoplace no)
-			(effects
-				(font
-					(size 1.27 1.27)
-				)
-			)
-		)
-		(property "Value" "+3.3V"
-			(at 107.95 76.2 0)
-			(show_name no)
-			(do_not_autoplace no)
-			(effects
-				(font
-					(size 1.27 1.27)
-				)
-			)
-		)
-		(property "Footprint" ""
-			(at 107.95 81.28 0)
-			(hide yes)
-			(show_name no)
-			(do_not_autoplace no)
-			(effects
-				(font
-					(size 1.27 1.27)
-				)
-			)
-		)
-		(property "Datasheet" ""
-			(at 107.95 81.28 0)
-			(hide yes)
-			(show_name no)
-			(do_not_autoplace no)
-			(effects
-				(font
-					(size 1.27 1.27)
-				)
-			)
-		)
-		(property "Description" "Power symbol creates a global label with name \"+3.3V\""
-			(at 107.95 81.28 0)
-			(hide yes)
-			(show_name no)
-			(do_not_autoplace no)
-			(effects
-				(font
-					(size 1.27 1.27)
-				)
-			)
-		)
-		(pin "1"
-		)
-		(instances
-			(project "PCB"
-				(path "/ce714510-8789-438c-9780-97c7c26e78af/77c81cbd-c586-4d65-a39c-d5337f0031c1"
-					(reference "#PWR0107")
 					(unit 1)
 				)
@@
 			)
 		)
-		(property "Value" "R-INMP441"
+		(property "Value" "L-INMP441"
 			(at 118.11 77.47 0)
 			(show_name no)

Commit message: [PCB] Splited the PCB into two boards
Connections:
- net +3.3V: no longer J17.1 (Pin_1)
- new net +3.3VCo: J17.1 (Pin_1)
Changed lines of the file:
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@@
 			)
 		)
-		(property "Value" "+3.3V"
-			(at 129.54 104.14 0)
+		(property "Value" "+3.3VCo"
+			(at 132.08 107.9499 0)
 			(show_name no)
 			(do_not_autoplace no)
@@
 					(size 1.27 1.27)
 				)
+				(justify left)
 			)
 		)
